File: 0031_Color_Module_TCS3200.kicad_sch (KiCad schematic)
At the start: 16 parts, among them U1 TCS3200

Commit message: Add files via upload
Parts:
- removed R2: 0r, symbol Device:R
- added D5: LED, LED_SMD:LED_0805_2012Metric, symbol Device:LED
- added R10: 470r, Resistor_SMD:R_0805_2012Metric, symbol Device:R
- added U2: ~, Moduler_:pin_header, symbol moduler_pin:air
- C1: footprint (none) -> Capacitor_SMD:C_0805_2012Metric
- C2: footprint (none) -> Capacitor_SMD:C_1206_3216Metric
- D1, D2, D3, D4: footprint (none) -> LED_THT:LED_D3.0mm
- R1, R3, R4, R5, R6, R7, R8: footprint (none) -> Resistor_SMD:R_0805_2012Metric
- R2: renamed from R9; footprint (none) -> Resistor_SMD:R_0805_2012Metric
- U1: footprint SOIC8 -> TCS3200:SOIC8
Connections:
- net GND: now also U1.4 (GND), D5.1 (K), U2.9
- net OE: now also U2.3
- net OUT: now also U2.16
- net S0: now also U2.1
- net S1: now also U2.2
- net S2: now also U2.17
- net S3: now also U2.18
- net VDD renamed +3V3
- net +3V3: now also R10.1, U2.8
- new net: D5.2 (A), R10.2
- no-connect marks 0 -> 10
Other:
- note added: "AIR PIN"
- note added: "SENSOR"
- moved on the sheet: C1, C2, D1, D2, D3, D4, R1, R2, R3, R4, R5, R6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
